File: pcb/clog-v3.kicad_sch (KiCad schematic)
At the start: 25 parts, among them J0 AudioJack4dpb, SW1 SW_Push, SW10 SW_Push, SW11 SW_Push, SW12 SW_Push, SW13 SW_Push, SW14 SW_Push, SW15 SW_Push, SW16 SW_Push, SW17 SW_Push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

Commit message: Update Reset Switch, Remove Holes From Plate
Parts:
- SW18, SW21: footprint footprints:reset-switch-4pin -> footprints:reset-switch-angled-4pin
Changed lines of the file:
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@@
     (property "Reference" "SW21" (id 0) (at 171.45 139.7 0))
     (property "Value" "SW_Push" (id 1) (at 171.45 142.24 0))
-    (property "Footprint" "footprints:reset-switch-4pin" (id 2) (at 171.45 142.24 0)
+    (property "Footprint" "footprints:reset-switch-angled-4pin" (id 2) (at 171.45 142.24 0)
       (effects (font (size 1.27 1.27)) hide)
     )
@@
     (property "Reference" "SW18" (id 0) (at 171.45 125.73 0))
     (property "Value" "SW_Push" (id 1) (at 171.45 128.27 0))
-    (property "Footprint" "footprints:reset-switch-4pin" (id 2) (at 171.45 128.27 0)
+    (property "Footprint" "footprints:reset-switch-angled-4pin" (id 2) (at 171.45 128.27 0)
       (effects (font (size 1.27 1.27)) hide)
     )
@@
     )
     (path "/4ec432be-e3b3-4d28-802c-33ca3fb66772"
-      (reference "SW18") (unit 1) (value "SW_Push") (footprint "footprints:reset-switch-4pin")
+      (reference "SW18") (unit 1) (value "SW_Push") (footprint "footprints:reset-switch-angled-4pin")
     )
     (path "/4f5b4d96-5a38-4b2e-a759-bc7d95440c8b"
@@
     )
     (path "/1d2751e3-008b-4ba0-af9e-dd39156435d8"
-      (reference "SW21") (unit 1) (value "SW_Push") (footprint "footprints:reset-switch-4pin")
+      (reference "SW21") (unit 1) (value "SW_Push") (footprint "footprints:reset-switch-angled-4pin")
     )
     (path "/c7a53cab-ad3a-43ee-8585-52abdf784d4b"
